File: lark-power.sch (KiCad schematic (older format))
At the start: 16 parts

Commit message: Finalize schematics and component selection
Remove SD interface
Rework power supplies
Parts:
- removed C? (x2): C, symbol C
- removed C?: CP, symbol CP
- removed D?: SK33, symbol 1N5819
- removed L?: 47uH, symbol INDUCTOR
- removed U?: LM2675M-5, Housings_SOIC:SOIC-8_3.9x4.9mm_Pitch1.27mm, symbol LM2675M-5
- added C11: 22u, Capacitors_SMD:C_1206_HandSoldering, symbol C
- added C12, C19: 1u, Capacitors_SMD:C_0805_HandSoldering, symbol C
- added C13, C14, C21: 100n, Capacitors_SMD:C_0805_HandSoldering, symbol C
- added C17: 10p, Capacitors_SMD:C_0805_HandSoldering, symbol C
- added C20: 10n, Capacitors_SMD:C_0805_HandSoldering, symbol C
- added D2: Transil, components:DO-214AA, symbol D_Schottky
- added L1: 2.2u, Inductors_NEOSID:Neosid_Inductor_SM-NE29_SMD1008, symbol INDUCTOR
- added R16: 18.2k, Resistors_SMD:R_0805_HandSoldering, symbol R
- added R17: 1M, Resistors_SMD:R_0805_HandSoldering, symbol R
- added R18: 187k, Resistors_SMD:R_0805_HandSoldering, symbol R
- added U3: LT8608, Housings_SSOP:MSOP-10-1EP_3x3mm_Pitch0.5mm, symbol LT8608
- C15: renamed from C?; value C -> 1u; footprint (none) -> Capacitors_SMD:C_0805_HandSoldering; PartNo (none) -> UMK212F105ZG-T
- C16: renamed from C?; value CP -> 220u; footprint (none) -> Capacitors_SMD:CP_Elec_8x10.5; PartNo (none) -> EEE1EA221UP
- C18, C23: renamed from C?; value C -> 100n; footprint (none) -> Capacitors_SMD:C_0805_HandSoldering; PartNo (none) -> 08055C104KAT2A
- C22: renamed from C?; value CP -> 22u; footprint (none) -> Capacitors_SMD:C_1206_HandSoldering; symbol CP -> C; PartNo (none) -> CL31A226KPHNNNE
- D3: renamed from D?; value MBR0560 -> Diode; footprint Diodes_SMD:SOD-123 -> Diodes_SMD:D_SOD-123; PartNo (none) -> MBR0560
- F1: renamed from F?; value F_Small -> PTGL; footprint (none) -> Varistors:RV_Disc_D9_W3.9_P5; PartNo (none) -> PTGL12AR1R2H2B51B0
- FB1: renamed from FB?; value FILTER -> Ferrite bead; footprint (none) -> Inductors_SMD:L_1206_Handsoldering; PartNo (none) -> BLM31KN121SN1L
- J4: renamed from J?; footprint (none) -> Connectors:AK300-2
- U4: renamed from U?; footprint (none) -> TO_SOT_Packages_SMD:SOT-223; PartNo (none) -> AZ1117CH-3.3TRG1DICT-ND
Connections:
- wire segments 36 -> 62
- no-connect marks 0 -> 2
Other:
- moved on the sheet: C15, C16, C18, D3, FB1
