File: lark-sensors.sch (KiCad schematic (older format))
At the start: 25 parts

Commit message: Finalize schematics and component selection
Remove SD interface
Rework power supplies
Parts:
- added C36, C37, C38, C39, C40, C41, C43: 100n, Capacitors_SMD:C_0805_HandSoldering, symbol C
- C24, C25, C26, C27, C28, C29, C30, C31, C32, C33, C34, C35: renamed from C?; value C -> 1u; footprint (none) -> Capacitors_SMD:C_0805_HandSoldering; PartNo (none) -> UMK212F105ZG-T
- C42: renamed from 100n; value C -> 100n; footprint (none) -> Capacitors_SMD:C_0805_HandSoldering; PartNo (none) -> 08055C104KAT2A
- IC1, IC2: renamed from IC?; footprint agg:MS5611 -> components:MS5611; PartNo (none) -> MS5611-01BA03
- L2, L3, L4, L5: renamed from L?; footprint (none) -> Inductors_SMD:L_0805_HandSoldering; PartNo (none) -> BLM21BD272SH1L
- U10: renamed from U?; footprint (none) -> components:SOIC-14W; PartNo (none) -> MS5525DSO
- U5, U6, U7, U8: renamed from U?; PartNo (none) -> MCP1700T-3302E/TT
- U9: renamed from U?; footprint (none) -> Housings_DFN_QFN:QFN-24-1EP_3x3mm_Pitch0.4mm; PartNo (none) -> MPU-9250
Connections:
- wire segments 110 -> 129

Commit message: Rework the schematic from scratch
Rework basic ESP32 pin assignment
Rework power supply
Rework interface
Rework sound generation - remove I2C codec, use internal DAC
Add D-class amplifier
Add Serial lines
Add USB charger
Parts:
- removed C24, C25, C26, C27, C28, C29, C30, C31, C32, C33, C34, C35: 1u, Capacitors_SMD:C_0805_HandSoldering, symbol C
- removed C36, C37, C38, C39, C40, C41, C42, C43: 100n, Capacitors_SMD:C_0805_HandSoldering, symbol C
- removed IC1, IC2: MS5611-01BA03, components:MS5611, symbol MS5611-01BA03
- removed L2, L3, L4, L5: INDUCTOR, Inductors_SMD:L_0805_HandSoldering, symbol INDUCTOR
- removed U10: MS5525DSO, components:SOIC-14W, symbol MS5525DSO
- removed U5, U6, U7, U8: MCP1700-3302E_SOT23, TO_SOT_Packages_SMD:SOT-23, symbol MCP1700-3302E_SOT23
- removed U9: MPU-9250, Housings_DFN_QFN:QFN-24-1EP_3x3mm_Pitch0.4mm, symbol MPU-9250
- added C? (x6): 100n, symbol Device:C
- added C? (x2): C, symbol Device:C
- added IC? (x2): MS5611-01BA03, agg:MS5611, symbol sensors:MS5611-01BA03
- added U?: MPU-9250, Package_DFN_QFN:QFN-24-1EP_3x3mm_P0.4mm_EP1.75x1.6mm, symbol Sensor_Motion:MPU-9250
- added U?: MS5525DSO, symbol sensors:MS5525DSO
Connections:
- net labels added: ACCELPWR, I2CCLK, I2CSDA, PDIFPWR, PDUSPWR, PSTATPWR, SPICLK, SPICS0, SPICS1, SPID, SPIQ
- net labels removed: +5V, CS0, CS1, I2C_CLK, I2C_SDA, MISO, MOSI, SCLK
- wire segments 129 -> 97

Commit message: Finalize schematic
Finish part selection

Pending issues: IMU, switches & LEDs, mechanical parts and housing
selection.
Parts:
- removed C?: 100n, symbol Device:C
- C33, C34, C36, C38, C39: renamed from C?; footprint (none) -> Capacitor_SMD:C_0805_2012Metric_Pad1.15x1.40mm_HandSolder; MPN (none) -> 885012207128
- C35, C37: renamed from C?; value C -> 100n; footprint (none) -> Capacitor_SMD:C_0805_2012Metric_Pad1.15x1.40mm_HandSolder; MPN (none) -> 885012207128
- IC1, IC2: renamed from IC?; footprint agg:MS5611 -> Package_LGA:LGA-8_3x5mm_P1.25mm; MPN (none) -> MS561101BA03-50
- U8: renamed from U?; MPN (none) -> MPU-9250
- U9: renamed from U?; footprint (none) -> Package_SO:SOIC-14W_7.5x9.0mm_P1.27mm; MPN (none) -> 5525DSO-DB001DS
Connections:
- net labels added: I2C0CLK, I2C0SDA, I2C1CLK, I2C1SDA
- net labels removed: I2CCLK, I2CSDA, SPICLK, SPICS0, SPICS1, SPID, SPIQ
- wire segments 97 -> 96
- no-connect marks 5 -> 6

Commit message: Replace MPU-9250 IMU with BMX055
Parts:
- removed C36: 100n, Capacitor_SMD:C_0805_2012Metric_Pad1.15x1.40mm_HandSolder, symbol Device:C
- removed U8: MPU-9250, Package_DFN_QFN:QFN-24-1EP_3x3mm_P0.4mm_EP1.75x1.6mm, symbol Sensor_Motion:MPU-9250
- added U8: BMX055, BMX055:BMX055, symbol bmx055:BMX055
- renumbered C37 to C36, C38 to C37, C39 to C38
Connections:
- wire segments 96 -> 100
- no-connect marks 6 -> 13
Other:
- moved on the sheet: C33, C34
Changed lines of the file:
@@
 $EndDescr
-$Comp
-L Sensor_Motion:MPU-9250 U8
-U 1 1 5C51A592
-P 8400 2750
-F 0 "U8" H 8650 1950 50  0000 C CNN
-F 1 "MPU-9250" H 8050 1950 50  0000 C CNN
-F 2 "Package_DFN_QFN:QFN-24-1EP_3x3mm_P0.4mm_EP1.75x1.6mm" H 8400 1750 50  0001 C CNN
-F 3 "https://store.invensense.com/datasheets/invensense/MPU9250REV1.0.pdf" H 8400 2600 50  0001 C CNN
-F 4 "MPU-9250" H 8400 2750 50  0001 C CNN "MPN"
-	1    8400 2750
-	1    0    0    -1
-$EndComp
 $Comp
 L sensors:MS5525DSO U9
@@
 	9250 5000 9000 5000
 $Comp
-L Device:C C39
+L Device:C C38
 U 1 1 5C572742
 P 10300 5550
-F 0 "C39" H 10415 5596 50  0000 L CNN
+F 0 "C38" H 10415 5596 50  0000 L CNN
 F 1 "100n" H 10415 5505 50  0000 L CNN
 F 2 "Capacitor_SMD:C_0805_2012Metric_Pad1.15x1.40mm_HandSolder" H 10338 5400 50  0001 C CNN
@@
 $EndComp
 $Comp
-L Device:C C38
+L Device:C C37
 U 1 1 5C572A29
 P 9600 5050
-F 0 "C38" H 9715 5096 50  0000 L CNN
+F 0 "C37" H 9715 5096 50  0000 L CNN
 F 1 "100n" H 9715 5005 50  0000 L CNN
 F 2 "Capacitor_SMD:C_0805_2012Metric_Pad1.15x1.40mm_HandSolder" H 9638 4900 50  0001 C CNN
@@
 $EndComp
 $Comp
-L Device:C C37
+L Device:C C36
 U 1 1 5C5741B1
 P 2950 4750
-F 0 "C37" H 3065 4796 50  0000 L CNN
+F 0 "C36" H 3065 4796 50  0000 L CNN
 F 1 "100n" H 3065 4705 50  0000 L CNN
 F 2 "Capacitor_SMD:C_0805_2012Metric_Pad1.15x1.40mm_HandSolder" H 2988 4600 50  0001 C CNN
@@
 Wire Wire Line
 	6050 2200 6050 2350
-Wire Wire Line
-	7700 2650 6050 2650
-Wire Wire Line
-	6050 2650 6050 2350
 Connection ~ 6050 2350
 $Comp
@@
 	1    0    0    -1
 $EndComp
-Wire Wire Line
-	7700 2950 7650 2950
-Wire Wire Line
-	7650 2950 7650 3850
-Wire Wire Line
-	7650 3850 8400 3850
-Wire Wire Line
-	8400 3650 8400 3850
-Connection ~ 8400 3850
 $Comp
 L Device:C C34
 U 1 1 5C593811
-P 8850 1600
-F 0 "C34" H 8965 1646 50  0000 L CNN
-F 1 "100n" H 8965 1555 50  0000 L CNN
-F 2 "Capacitor_SMD:C_0805_2012Metric_Pad1.15x1.40mm_HandSolder" H 8888 1450 50  0001 C CNN
-F 3 "~" H 8850 1600 50  0001 C CNN
-F 4 "885012207128" H 8850 1600 50  0001 C CNN "MPN"
-	1    8850 1600
+P 9200 1600
+F 0 "C34" H 9315 1646 50  0000 L CNN
+F 1 "100n" H 9315 1555 50  0000 L CNN
+F 2 "Capacitor_SMD:C_0805_2012Metric_Pad1.15x1.40mm_HandSolder" H 9238 1450 50  0001 C CNN
+F 3 "~" H 9200 1600 50  0001 C CNN
+F 4 "885012207128" H 9200 1600 50  0001 C CNN "MPN"
+	1    9200 1600
 	1    0    0    -1
 $EndComp
@@
 L Device:C C33
 U 1 1 5C593886
-P 7950 1600
-F 0 "C33" H 8065 1646 50  0000 L CNN
-F 1 "100n" H 8065 1555 50  0000 L CNN
-F 2 "Capacitor_SMD:C_0805_2012Metric_Pad1.15x1.40mm_HandSolder" H 7988 1450 50  0001 C CNN
-F 3 "~" H 7950 1600 50  0001 C CNN
-F 4 "885012207128" H 7950 1600 50  0001 C CNN "MPN"
-	1    7950 1600
-	1    0    0    -1
-$EndComp
-Text HLabel 8300 1350 1    50   Input ~ 0
+P 7850 1600
+F 0 "C33" H 7965 1646 50  0000 L CNN
+F 1 "100n" H 7965 1555 50  0000 L CNN
+F 2 "Capacitor_SMD:C_0805_2012Metric_Pad1.15x1.40mm_HandSolder" H 7888 1450 50  0001 C CNN
+F 3 "~" H 7850 1600 50  0001 C CNN
+F 4 "885012207128" H 7850 1600 50  0001 C CNN "MPN"
+	1    7850 1600
+	1    0    0    -1
+$EndComp
+Text HLabel 8600 1300 1    50   Input ~ 0
 ACCELPWR
-Wire Wire Line
-	8300 1350 8300 1400
-Wire Wire Line
-	8300 1400 7950 1400
-Wire Wire Line
-	7950 1400 7950 1450
-Wire Wire Line
-	8300 1400 8500 1400
-Wire Wire Line
-	8850 1400 8850 1450
-Connection ~ 8300 1400
-Wire Wire Line
-	8500 1850 8500 1400
-Connection ~ 8500 1400
-Wire Wire Line
-	8500 1400 8850 1400
-Wire Wire Line
-	8300 1400 8300 1850
 $Comp
 L power:GND #PWR036
 U 1 1 5C59D0F5
-P 8850 1800
-F 0 "#PWR036" H 8850 1550 50  0001 C CNN
-F 1 "GND" H 8855 1627 50  0000 C CNN
-F 2 "" H 8850 1800 50  0001 C CNN
-F 3 "" H 8850 1800 50  0001 C CNN
-	1    8850 1800
+P 9200 1800
+F 0 "#PWR036" H 9200 1550 50  0001 C CNN
+F 1 "GND" H 9205 1627 50  0000 C CNN
+F 2 "" H 9200 1800 50  0001 C CNN
+F 3 "" H 9200 1800 50  0001 C CNN
+	1    9200 1800
 	1    0    0    -1
 $EndComp
@@
 L power:GND #PWR035
 U 1 1 5C59D1AD
-P 7950 1800
-F 0 "#PWR035" H 7950 1550 50  0001 C CNN
-F 1 "GND" H 7955 1627 50  0000 C CNN
-F 2 "" H 7950 1800 50  0001 C CNN
-F 3 "" H 7950 1800 50  0001 C CNN
-	1    7950 1800
-	1    0    0    -1
-$EndComp
-Wire Wire Line
-	8850 1750 8850 1800
-Wire Wire Line
-	7950 1800 7950 1750
-$Comp
-L Device:C C36
-U 1 1 5C5A22FB
-P 9600 3100
-F 0 "C36" H 9715 3146 50  0000 L CNN
-F 1 "100n" H 9715 3055 50  0000 L CNN
-F 2 "Capacitor_SMD:C_0805_2012Metric_Pad1.15x1.40mm_HandSolder" H 9638 2950 50  0001 C CNN
-F 3 "~" H 9600 3100 50  0001 C CNN
-F 4 "885012207128" H 9600 3100 50  0001 C CNN "MPN"
-	1    9600 3100
-	1    0    0    -1
-$EndComp
-Wire Wire Line
-	9100 3050 9300 3050
-Wire Wire Line
-	9300 3050 9300 1400
-Wire Wire Line
-	9300 1400 8850 1400
-Connection ~ 8850 1400
-Wire Wire Line
-	9100 2950 9600 2950
-Wire Wire Line
-	9100 3150 9200 3150
-Wire Wire Line
-	9200 3850 8400 3850
-Wire Wire Line
-	9600 3250 9600 3850
-Wire Wire Line
-	9600 3850 9200 3850
-Connection ~ 9200 3850
-NoConn ~ 9100 2750
-NoConn ~ 9100 2650
-NoConn ~ 9100 2450
+P 7850 1800
+F 0 "#PWR035" H 7850 1550 50  0001 C CNN
+F 1 "GND" H 7855 1627 50  0000 C CNN
+F 2 "" H 7850 1800 50  0001 C CNN
+F 3 "" H 7850 1800 50  0001 C CNN
+	1    7850 1800
+	1    0    0    -1
+$EndComp
 Wire Wire Line
 	4450 2350 6050 2350
@@
 	10300 5800 10300 5900
 Wire Wire Line
-	9200 3150 9200 3850
-Wire Wire Line
 	3500 2550 3500 2650
 Wire Wire Line
@@
 NoConn ~ 4450 2550
 Wire Wire Line
-	7700 2550 7650 2550
-Wire Wire Line
-	7650 2550 7650 2950
-Connection ~ 7650 2950
-Wire Wire Line
 	6150 2200 6150 2450
+$Comp
+L bmx055:BMX055 U8
+U 1 1 5C6812A2
+P 8500 2800
+F 0 "U8" H 8525 3765 50  0000 C CNN
+F 1 "BMX055" H 8525 3674 50  0000 C CNN
+F 2 "BMX055:BMX055" H 8600 2800 50  0001 C CNN
+F 3 "" H 8600 2800 50  0001 C CNN
+F 4 "828-1060-1-ND " H 8500 2800 50  0001 C CNN "MPN"
+	1    8500 2800
+	1    0    0    -1
+$EndComp
+Wire Wire Line
+	8400 3850 9600 3850
+NoConn ~ 9350 2450
+NoConn ~ 9350 2300
+NoConn ~ 7700 2750
+NoConn ~ 7700 3200
+NoConn ~ 7700 3500
+NoConn ~ 9350 2750
+Wire Wire Line
+	9350 3500 9400 3500
+Wire Wire Line
+	9400 3500 9400 4200
+Wire Wire Line
+	7000 2350 6050 2350
+Wire Wire Line
+	6900 2450 6150 2450
 Connection ~ 6150 2450
 Wire Wire Line
-	6150 2450 7700 2450
-Wire Wire Line
-	7700 2750 7550 2750
-Wire Wire Line
-	7550 2750 7550 1400
-Wire Wire Line
-	7550 1400 7950 1400
-Connection ~ 7950 1400
+	6900 2450 6900 4200
+Wire Wire Line
+	6900 4200 9400 4200
+Wire Wire Line
+	7000 2350 7000 3350
+Wire Wire Line
+	7000 3350 7700 3350
+Wire Wire Line
+	9600 2150 9350 2150
+Wire Wire Line
+	9600 2150 9600 2600
+Wire Wire Line
+	9350 3350 9600 3350
+Connection ~ 9600 3350
+Wire Wire Line
+	9600 3350 9600 3850
+Wire Wire Line
+	9350 2600 9600 2600
+Connection ~ 9600 2600
+Wire Wire Line
+	9600 2600 9600 3350
+Wire Wire Line
+	9350 3200 9700 3200
+Wire Wire Line
+	9700 3200 9700 1400
+Wire Wire Line
+	7700 2450 7500 2450
+Wire Wire Line
+	7500 2450 7500 1400
+NoConn ~ 9350 2900
+NoConn ~ 9350 3050
+NoConn ~ 7700 2150
+NoConn ~ 7700 2300
+Wire Wire Line
+	7500 2450 7500 3050
+Wire Wire Line
+	7500 3050 7700 3050
+Connection ~ 7500 2450
+Wire Wire Line
+	7700 2600 7400 2600
+Wire Wire Line
+	7400 2600 7400 2900
+Wire Wire Line
+	7400 3850 8400 3850
+Connection ~ 8400 3850
+Wire Wire Line
+	7700 2900 7400 2900
+Connection ~ 7400 2900
+Wire Wire Line
+	7400 2900 7400 3850
+Wire Wire Line
+	7500 1400 7850 1400
+Wire Wire Line
+	7850 1450 7850 1400
+Connection ~ 7850 1400
+Wire Wire Line
+	7850 1800 7850 1750
+Wire Wire Line
+	9200 1450 9200 1400
+Connection ~ 9200 1400
+Wire Wire Line
+	9200 1400 9700 1400
+Wire Wire Line
+	9200 1750 9200 1800
+Wire Wire Line
+	7850 1400 8600 1400
+Wire Wire Line
+	8600 1300 8600 1400
+Connection ~ 8600 1400
+Wire Wire Line
+	8600 1400 9200 1400
 $EndSCHEMATC

Commit message: Intermediate status while arranging compontents.
Manually grouped components into smaller islands.

Some parts were changed:
* U1: SOT-23-3 LDO should be sufficient
* CP_Elec: Use 10x10 size
Parts:
- U8: symbol bmx055:BMX055 -> lark-rescue:BMX055-bmx055
Connections:
- wire segments 100 -> 98
Changed lines of the file:
@@
 	3750 4900 3500 4900
 Connection ~ 3500 4900
-Wire Wire Line
-	3500 4900 3500 5050
-Wire Wire Line
-	4450 4900 4500 4900
-Wire Wire Line
-	4500 4900 4500 5050
-Wire Wire Line
-	4500 5050 3500 5050
-Connection ~ 3500 5050
-Wire Wire Line
-	3500 5050 3500 5100
 NoConn ~ 4450 4800
 Wire Wire Line
@@
 	4500 2650 4450 2650
 Wire Wire Line
-	7800 5300 6250 5300
-Wire Wire Line
-	6250 5300 6250 4700
-Wire Wire Line
-	6250 4700 4450 4700
-Wire Wire Line
-	7800 5400 6150 5400
-Wire Wire Line
-	6150 5400 6150 4600
-Text HLabel 6150 4400 1    50   Input ~ 0
+	7800 5300 7100 5300
+Wire Wire Line
+	7800 5400 7000 5400
+Text HLabel 5400 2150 1    50   Input ~ 0
 I2C0CLK
 Wire Wire Line
-	6150 4400 6150 4600
-Connection ~ 6150 4600
-Text HLabel 6250 4400 1    50   Input ~ 0
+	5400 2150 5400 2350
+Text HLabel 5500 2150 1    50   Input ~ 0
 I2C0SDA
 Wire Wire Line
-	6250 4400 6250 4700
-Wire Wire Line
-	4450 4600 6150 4600
-Connection ~ 6250 4700
-Text HLabel 6150 2200 1    50   Input ~ 0
+	5500 2150 5500 2450
+Wire Wire Line
+	4450 4600 5400 4600
+Text HLabel 7100 2200 1    50   Input ~ 0
 I2C1SDA
-Text HLabel 6050 2200 1    50   Input ~ 0
+Text HLabel 7000 2200 1    50   Input ~ 0
 I2C1CLK
-Wire Wire Line
-	6050 2200 6050 2350
-Connection ~ 6050 2350
 $Comp
 L power:GND #PWR038
@@
 $EndComp
 Wire Wire Line
-	4450 2350 6050 2350
-Wire Wire Line
 	9600 4900 10300 4900
 Wire Wire Line
@@
 Wire Wire Line
 	3500 2350 2950 2350
-Wire Wire Line
-	4450 2450 6150 2450
 NoConn ~ 4450 2550
-Wire Wire Line
-	6150 2200 6150 2450
-$Comp
-L bmx055:BMX055 U8
+$Comp
+L lark-rescue:BMX055-bmx055 U8
 U 1 1 5C6812A2
 P 8500 2800
+AR Path="/5C6812A2" Ref="U8"  Part="1"
+AR Path="/5C4F6DA1/5C6812A2" Ref="U8"  Part="1"
 F 0 "U8" H 8525 3765 50  0000 C CNN
 F 1 "BMX055" H 8525 3674 50  0000 C CNN
@@
 	9400 3500 9400 4200
 Wire Wire Line
-	7000 2350 6050 2350
-Wire Wire Line
-	6900 2450 6150 2450
-Connection ~ 6150 2450
-Wire Wire Line
-	6900 2450 6900 4200
-Wire Wire Line
-	6900 4200 9400 4200
-Wire Wire Line
-	7000 2350 7000 3350
+	7100 4200 9400 4200
 Wire Wire Line
 	7000 3350 7700 3350
@@
 Wire Wire Line
 	8600 1400 9200 1400
+Wire Wire Line
+	4450 2350 5400 2350
+Wire Wire Line
+	4450 2450 5500 2450
+Wire Wire Line
+	5500 4700 4450 4700
+Wire Wire Line
+	3500 4900 3500 5100
+Wire Wire Line
+	4600 4900 4600 4450
+Wire Wire Line
+	4600 4450 3500 4450
+Wire Wire Line
+	3500 4450 3500 4600
+Wire Wire Line
+	4450 4900 4600 4900
+Wire Wire Line
+	5400 2350 5400 4600
+Wire Wire Line
+	5500 2450 5500 4700
+Wire Wire Line
+	7100 2200 7100 4200
+Wire Wire Line
+	7000 2200 7000 3350
+Connection ~ 7000 3350
+Connection ~ 7100 4200
+Wire Wire Line
+	7100 4200 7100 5300
+Wire Wire Line
+	7000 3350 7000 5400
+Connection ~ 5400 2350
+Connection ~ 5500 2450
 $EndSCHEMATC

Commit message: continue layout work, WIP
Parts:
- C33, C34, C35, C36, C37, C38: symbol Device:C -> lark-rescue:C-Device
Changed lines of the file:
@@
 	9250 5000 9000 5000
 $Comp
-L Device:C C38
+L lark-rescue:C-Device C38
 U 1 1 5C572742
 P 10300 5550
@@
 $EndComp
 $Comp
-L Device:C C37
+L lark-rescue:C-Device C37
 U 1 1 5C572A29
 P 9600 5050
@@
 	9350 5100 9000 5100
 $Comp
-L power:GND #PWR041
+L lark-rescue:GND-power #PWR041
 U 1 1 5C5732B7
 P 10300 5900
@@
 	9350 5400 9350 5200
 $Comp
-L power:GND #PWR040
+L lark-rescue:GND-power #PWR040
 U 1 1 5C5738F4
 P 9150 5600
@@
 NoConn ~ 7800 5200
 $Comp
-L Device:C C35
+L lark-rescue:C-Device C35
 U 1 1 5C5740F5
 P 2950 2500
@@
 $EndComp
 $Comp
-L Device:C C36
+L lark-rescue:C-Device C36
 U 1 1 5C5741B1
 P 2950 4750
@@
 	3500 4600 3750 4600
 $Comp
-L power:GND #PWR039
+L lark-rescue:GND-power #PWR039
 U 1 1 5C575803
 P 3500 5100
@@
 $EndComp
 $Comp
-L power:GND #PWR037
+L lark-rescue:GND-power #PWR037
 U 1 1 5C5758C5
 P 3500 3000
@@
 I2C1CLK
 $Comp
-L power:GND #PWR038
+L lark-rescue:GND-power #PWR038
 U 1 1 5C58F414
 P 8400 3850
@@
 $EndComp
 $Comp
-L Device:C C34
+L lark-rescue:C-Device C34
 U 1 1 5C593811
 P 9200 1600
@@
 $EndComp
 $Comp
-L Device:C C33
+L lark-rescue:C-Device C33
 U 1 1 5C593886
 P 7850 1600
@@
 ACCELPWR
 $Comp
-L power:GND #PWR036
+L lark-rescue:GND-power #PWR036
 U 1 1 5C59D0F5
 P 9200 1800
@@
 $EndComp
 $Comp
-L power:GND #PWR035
+L lark-rescue:GND-power #PWR035
 U 1 1 5C59D1AD
 P 7850 1800
