File: lark.kicad_pcb (KiCad board)
At the start: 2 copper layers, 137.5 x 51 mm, 109 parts, among them CON1 SJ1-3523N, IC1 MS5611-01BA03, IC2 MS5611-01BA03, IC3 BMP388, IC4 BMP388, J1 CONN1, J10 Conn_01x05-Connector_Generic, J11 CONN1, J2 Conn_01x05-Connector_Generic, J3 Conn_01x05-Connector_Generic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

Commit message: update layout
IRQs connected
somehow handsoldering friendly BS5611

DRC is OK.
Unconnected: 5 nets (will later connect the sensor board)
Parts:
- added R3: 100k, Resistor_SMD:R_0805_2012Metric_Pad1.15x1.40mm_HandSolder, F.Cu at (175.4, 121.0)
- added R4: 1k, Resistor_SMD:R_0805_2012Metric_Pad1.15x1.40mm_HandSolder, F.Cu at (182.7, 130.0)
- added R5: 1k, Resistor_SMD:R_0805_2012Metric_Pad1.15x1.40mm_HandSolder, F.Cu at (180.4, 130.0)
- IC1, IC2: footprint Package_LGA:LGA-8_3x5mm_P1.25mm -> libs:LGA-8_3x5mm_P1.25mm_handsolder
- moved C1 0.70 mm to (157.4, 130.7)
- moved R2 0.70 mm to (159.4, 130.7)
Connections:
- J3 pad 2: Net-(J3-Pad2) -> INT_SENS
- J5 pad 2: Net-(J5-Pad2) -> Net-(J2-Pad2)
- MOD1 pad 12: INT_GYR -> INT_IMU
- MOD1 pad 13: INT_ACC -> INT_SENS
- U5 pad 17: Net-(U5-Pad17) -> Net-(J2-Pad2)
- U5 pad 4: /Sensors/SENSPWR -> Net-(IC3-Pad7)
- U5 pad 7: /Sensors/SENSPWR -> Net-(IC4-Pad7)
- U6 pad 12: INT_GYR -> Net-(R5-Pad2)
- U6 pad 16: INT_ACC -> Net-(R4-Pad2)
Routing:
- net INT_SENS: track 0.00 -> 68.3 mm, vias 0 -> 2
- net Net-(J2-Pad2): track 0.00 -> 50.2 mm, vias 0 -> 1
- net INT_IMU: track 0.00 -> 40.4 mm, vias 0 -> 3
- net INT_ACC: track 36.4 -> 0.00 mm, vias 2 -> 0
- net INT_GYR: track 35.7 -> 0.00 mm, vias 2 -> 0
- net Net-(IC3-Pad7): track 0.00 -> 23.8 mm, vias 0 -> 1
- net Net-(IC4-Pad7): track 0.00 -> 22.0 mm, vias 0 -> 1
- net /Sensors/SENSPWR: track 216.4 -> 209.9 mm
- net Net-(R5-Pad2): track 0.00 -> 4.88 mm
- net /Power/ACCELPWR: track 11.9 -> 15.8 mm
- net Net-(R4-Pad2): track 0.00 -> 2.52 mm
- net GND: track 22.9 -> 24.3 mm, vias 87 -> 86
- net SND_R: track 24.0 -> 25.0 mm
- net /Sensors/SDA0: track 48.1 -> 48.8 mm
